File: QL_MiniTrump3.kicad_pcb (KiCad board)
At the start: 2 copper layers, 73 x 99.1 mm, 25 parts, among them J1 QL_SLOT_DIN41612_CARD, J2 Conn_02x17_Odd_Even, J3 QL_SLOT_DIN41612_CARD, U1 GAL16V8, U14 27C128, U15 74HC04, U17 74ls175, U18 7805, X1 CXO_DIP8

Commit message: Rev 2, with GAL code
Parts:
- added JP1: Jumper_2_Open, Jumper:SolderJumper-2_P1.3mm_Open_RoundedPad1.0x1.5mm, B.Cu at (181.8, 101.5)
- C1, C10, C12, C13, C15, C2, C3, C4: value C -> 100n
- C14, C16: value C_Polarized -> 100uF/16V
- D1, D6, D7, D8: footprint Diode_SMD:D_1206_3216Metric -> Diode_SMD:D_0805_2012Metric
- J1: value QL_SLOT_DIN41612_CARD -> QL_SLOT_DIN41612F
- J3: value QL_SLOT_DIN41612_CARD -> QL_SLOT_DIN41612M
- U17: value 74ls175 -> 74LS175
- X1: value CXO_DIP8 -> 8Mhz
- renumbered U to U13
Connections:
- J1 pad a4: /SP0 -> +5V
- J1 pad b28: unconnected-(J1-~{AS}-Padb28) -> /AS
- J1 pad b5: unconnected-(J1-~{BERR}-Padb5) -> Net-(J1-~{BERR})
- J3 pad b28: unconnected-(J3-~{AS}-Padb28) -> /AS
- U1 pad 13: unconnected-(U1-IO7-Pad13) -> /P13
Routing:
- net Net-(J1-~{BERR}): track 0.00 -> 121.4 mm
- net /AS: track 0.00 -> 72.6 mm, vias 0 -> 2
- net /SP0: track 67.5 -> 0.00 mm
- net +5V: track 183.8 -> 201.8 mm
- net /A18: track 99.0 -> 88.8 mm
- net /P13: track 0.00 -> 2.55 mm
- net /D6: track 109.4 -> 111.6 mm
- net /SP1: track 70.0 -> 71.7 mm
- net /D5: track 112.5 -> 114.2 mm
- net /DTACKL: track 79.2 -> 80.7 mm
- net /CS175: track 32.2 -> 33.4 mm
- net /D4: track 125.6 -> 126.7 mm
- net /DS: track 72.8 -> 73.8 mm
- net /D0: track 154.8 -> 155.7 mm
- net /A14: track 97.6 -> 98.4 mm
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Other:
- board text added: "Rev. 2"
